Commit message: 20241126

File: support/ros_industrial_support/urdf/robot_pedestal/robot1_pedestal.xacro (robot description, xacro)
@@ -5,5 +5,4 @@
   <xacro:arg name="pedestal_height" default="0.95"/>
   <link name="world_interface"/>
-  <!-- URDF -->
   <xacro:include filename="$(find ros_industrial_support)/urdf/robot_pedestal/robot_pedestal.urdf.xacro"/>
   <xacro:robot_pedestal_urdf pedestal_prefix="$(arg pedestal_prefix)" pedestal_parent="$(arg pedestal_parent)" pedestal_height="$(arg pedestal_height)">

File: support/ros_industrial_support/urdf/robot_pedestal/robot_pedestal.urdf.xacro (robot description, xacro)
@@ -3,6 +3,8 @@
 <!-- robot pedestal -->
 <xacro:macro name = "robot_pedestal_urdf" params = "pedestal_prefix pedestal_parent pedestal_height *origin">
-  <joint name="${pedestal_prefix}pedestal_joint" type="fixed">
+  <joint name="${pedestal_prefix}_pedestal_joint" type="fixed">
+    <!--
     <xacro:insert_block name="origin" />
+    -->
     <parent link="${pedestal_parent}"/>
     <child link="${pedestal_prefix}pedestal_link"/>
