Commit message: 20241128

File: support/ros_industrial_support/urdf/bin/bin.urdf.xacro (robot description, xacro)
@@ -1,5 +1,7 @@
 <?xml version="1.0"?>
 <robot xmlns:xacro="http://www.ros.org/wiki/xacro">
-  <xacro:macro name="bin_urdf" params="prefix mesh_path:='package://ros_industrial_support'">
+  <xacro:arg name="mesh_path" default="$(find ros_industrial_support)"/>
+  <!--<xacro:macro name="bin_urdf" params="prefix mesh_path:='package://ros_industrial_support'">-->
+  <xacro:macro name="bin_urdf" params="prefix">
     <!-- link list -->
     <link name="${prefix}base_link">
@@ -7,5 +9,6 @@
         <origin xyz="0 0 0" rpy="0 0 0" />
         <geometry>
-          <mesh filename="${mesh_path}/meshes/bin/visual/bin.dae" />
+          <mesh filename="$(find ros_industrial_support)/meshes/bin/visual/bin.dae" />
+          <mesh filename="package://ros_industrial_support/meshes/bin/visual/bin.dae" />
           <scale>0.6 0.6 0.6</scale>
         </geometry>
@@ -14,5 +17,5 @@
         <origin xyz="0 0 0" rpy="0 0 0"/>
         <geometry>
-          <mesh filename="${mesh_path}/meshes/bin/collision/bin_bottom.dae"/>
+          <mesh filename="$(find ros_industrial_support)/meshes/bin/collision/bin_bottom.dae"/>
           <scale>0.6 0.6 0.6</scale>
         </geometry>
@@ -21,5 +24,5 @@
         <origin xyz="0 0 0" rpy="0 0 0"/>
         <geometry>
-          <mesh filename="${mesh_path}/meshes/bin/collision/bin_sides.dae"/>
+          <mesh filename="$(find ros_industrial_support)/meshes/bin/collision/bin_sides.dae"/>
           <scale>0.6 0.6 0.6</scale>
         </geometry>
