Commit message: 20241127

File: 5_transferframes/transferframes/urdf/environment.urdf.xacro (robot description, xacro)
@@ -26,5 +26,5 @@
  <!-- Robot1 -->
   <xacro:include filename="$(find ros_industrial_support)/urdf/ufactory/ufactory_xarm6.urdf.xacro"/>
-  <xacro:ufactory_xarm6 prefix="robot1_" joint_limited="true"/>
+  <xacro:ufactory_xarm6 prefix="" joint_limited="true"/>
   <!-- Vacuum Gripper1 -->
   <xacro:include filename="$(find ros_industrial_support)/urdf/vacuum_gripper/vacuum_gripper.urdf.xacro"/>
@@ -32,4 +32,7 @@
   <!-- bins -->
   <xacro:include filename="$(find ros_industrial_support)/urdf/bin/bin.urdf.xacro"/>
+  <!--
+  <xacro:bin_urdf prefix="bin_1_" mesh_path="package://ros_industrial_support"/>
+  -->
   <xacro:bin_urdf prefix="bin_1_"/>
   <!-- bin to world. -->
@@ -43,9 +46,9 @@
     <origin xyz="0 0 1.15" rpy="0 0 ${radians(0)}" />
     <parent link="robot1_pedestal_link" />
-    <child link="robot1_base_link" />
+    <child link="base_link" />
   </joint>
   <!-- gripper1 to robot1. -->
   <joint name="gripper1_to_robot1" type="fixed">
-    <parent link="robot1_tool_link" />
+    <parent link="tool_link" />
     <child link="vacuum_gripper1_base_link" />
   </joint>

File: support/ros_industrial_support/urdf/assembly_station/assembly_station.urdf.xacro (robot description, xacro)
@@ -1,5 +1,5 @@
 <?xml version="1.0" ?>
 <robot name="assembly_station_urdf" xmlns:xacro="http://www.ros.org/wiki/xacro">
-    <xacro:macro name="assembly_station_urdf" params="assembly_station_parent assembly_station_prefix *origin">
+    <xacro:macro name="assembly_station_urdf" params="assembly_station_parent assembly_station_prefix mesh_path:='package://ros_industrial_support' *origin">
   <joint name="${assembly_station_prefix}joint" type="fixed">
     <xacro:insert_block name="origin" />
@@ -14,10 +14,10 @@
       <visual>
         <geometry>
-          <mesh filename="package://ros_industrial_support/meshes/assembly_station/meshes/assembly_station.dae" scale="1.1 1.1 1.1"/>
+          <mesh filename="${mesh_path}/meshes/assembly_station/meshes/assembly_station.dae" scale="1.1 1.1 1.1"/>
         </geometry>
       </visual>
       <collision>
         <geometry>
-          <mesh filename="package://ros_industrial_support/meshes/assembly_station/meshes/assembly_station.dae" scale="1.1 1.1 1.1"/>
+          <mesh filename="${mesh_path}/meshes/assembly_station/meshes/assembly_station.dae" scale="1.1 1.1 1.1"/>
         </geometry>
       </collision>

File: support/ros_industrial_support/urdf/assembly_station/assembly_station.xacro (robot description, xacro)
@@ -3,4 +3,5 @@
   <xacro:arg name="assembly_station_prefix" default="assembly_station_"/>
   <xacro:arg name="assembly_station_parent" default="world_interface"/>
+  <xacro:arg name="mesh_path" default="$(find ros_industrial_support)"/>
   <xacro:arg name="x" default="0"/>
   <xacro:arg name="y" default="0"/>
@@ -12,5 +13,5 @@
   <!-- URDF -->
   <xacro:include filename="$(find ros_industrial_support)/urdf/assembly_station/assembly_station.urdf.xacro"/>
-  <xacro:assembly_station_urdf assembly_station_prefix="$(arg assembly_station_prefix)" assembly_station_parent="$(arg assembly_station_parent)">
+  <xacro:assembly_station_urdf assembly_station_prefix="$(arg assembly_station_prefix)" assembly_station_parent="$(arg assembly_station_parent)" mesh_path="$(arg mesh_path)">
      <origin xyz="$(arg x) $(arg y) $(arg z)" rpy="$(arg R) $(arg P) $(arg Y)"/>
   </xacro:assembly_station_urdf>

File: support/ros_industrial_support/urdf/bin/bin.urdf.xacro (robot description, xacro)
@@ -1,5 +1,5 @@
 <?xml version="1.0"?>
 <robot xmlns:xacro="http://www.ros.org/wiki/xacro">
-  <xacro:macro name="bin_urdf" params="prefix">
+  <xacro:macro name="bin_urdf" params="prefix mesh_path:='package://ros_industrial_support'">
     <!-- link list -->
     <link name="${prefix}base_link">
@@ -7,5 +7,5 @@
         <origin xyz="0 0 0" rpy="0 0 0" />
         <geometry>
-          <mesh filename="package://ros_industrial_support/meshes/bin/visual/bin.dae" />
+          <mesh filename="${mesh_path}/meshes/bin/visual/bin.dae" />
           <scale>0.6 0.6 0.6</scale>
         </geometry>
@@ -14,5 +14,5 @@
         <origin xyz="0 0 0" rpy="0 0 0"/>
         <geometry>
-          <mesh filename="package://ros_industrial_support/meshes/bin/collision/bin_bottom.dae"/>
+          <mesh filename="${mesh_path}/meshes/bin/collision/bin_bottom.dae"/>
           <scale>0.6 0.6 0.6</scale>
         </geometry>
@@ -21,5 +21,5 @@
         <origin xyz="0 0 0" rpy="0 0 0"/>
         <geometry>
-          <mesh filename="package://ros_industrial_support/meshes/bin/collision/bin_sides.dae"/>
+          <mesh filename="${mesh_path}/meshes/bin/collision/bin_sides.dae"/>
           <scale>0.6 0.6 0.6</scale>
         </geometry>

File: support/ros_industrial_support/urdf/bin/bin.xacro (robot description, xacro)
@@ -2,7 +2,11 @@
 <robot name="bin" xmlns:xacro="http://www.ros.org/wiki/xacro">
   <xacro:arg name="prefix" default="bin_1_"/>
+  <!--
+  <xacro:arg name="mesh_path" default="package://ros_industrial_support"/>
+  -->
+  <xacro:arg name="mesh_path" default="$(find ros_industrial_support)"/>
   <!-- URDF -->
   <xacro:include filename="$(find ros_industrial_support)/urdf/bin/bin.urdf.xacro"/>
-  <xacro:bin_urdf prefix="$(arg prefix)"/>
+  <xacro:bin_urdf prefix="$(arg prefix)" mesh_path="$(arg mesh_path)"/>
   <!-- Gazebo -->
   <xacro:include filename="$(find ros_industrial_support)/urdf/bin/bin.gazebo.xacro"/>

File: support/ros_industrial_support/urdf/computer_mobile/computer.urdf.xacro (robot description, xacro)
@@ -1,5 +1,5 @@
 <?xml version="1.0" ?>
 <robot name="computer_urdf" xmlns:xacro="http://www.ros.org/wiki/xacro">
-    <xacro:macro name="computer_urdf" params="computer_parent computer_prefix *origin">
+    <xacro:macro name="computer_urdf" params="computer_parent computer_prefix mesh_path:='package://ros_industrial_support' *origin">
   <joint name="${computer_prefix}joint" type="fixed">
     <xacro:insert_block name="origin" />
@@ -14,10 +14,10 @@
       <visual>
         <geometry>
-          <mesh filename="package://ros_industrial_support/meshes/computer_mobile/meshes/computer.dae" scale="0.01 0.01 0.01"/>
+          <mesh filename="${mesh_path}/meshes/computer_mobile/meshes/computer.dae" scale="0.01 0.01 0.01"/>
         </geometry>
       </visual>
       <collision>
         <geometry>
-          <mesh filename="package://ros_industrial_support/meshes/computer_mobile/meshes/computer.dae" scale="0.01 0.01 0.01"/>
+          <mesh filename="${mesh_path}/meshes/computer_mobile/meshes/computer.dae" scale="0.01 0.01 0.01"/>
         </geometry>
       </collision>

File: support/ros_industrial_support/urdf/computer_mobile/computer.xacro (robot description, xacro)
@@ -3,4 +3,5 @@
   <xacro:arg name="computer_prefix" default="computer_"/>
   <xacro:arg name="computer_parent" default="world_interface"/>
+  <xacro:arg name="mesh_path" default="$(find ros_industrial_support)"/>
   <xacro:arg name="x" default="0"/>
   <xacro:arg name="y" default="0"/>
@@ -12,5 +13,5 @@
   <!-- URDF -->
   <xacro:include filename="$(find ros_industrial_support)/urdf/computer_mobile/computer.urdf.xacro"/>
-  <xacro:computer_urdf computer_prefix="$(arg computer_prefix)" computer_parent="$(arg computer_parent)">
+  <xacro:computer_urdf computer_prefix="$(arg computer_prefix)" computer_parent="$(arg computer_parent)" mesh_path ="$(arg mesh_path)">
      <origin xyz="$(arg x) $(arg y) $(arg z)" rpy="$(arg R) $(arg P) $(arg Y)"/>
   </xacro:computer_urdf>

Commit message: 20241130

File: 5_transferframes/transferframes/urdf/environment.urdf.xacro (robot description, xacro)
@@ -11,5 +11,5 @@
   -->
   <xacro:include filename="$(find ros_industrial_support)/urdf/assembly_station/assembly_station.urdf.xacro"/>
-  <xacro:assembly_station_urdf assembly_station_prefix="shelf_" assembly_station_parent="world">
+  <xacro:assembly_station_urdf assembly_station_prefix="assembly_station_" assembly_station_parent="world">
     <origin xyz="0.5 -0.5 0.0" rpy="0 0 ${radians(90)}"/>
   </xacro:assembly_station_urdf>
@@ -17,5 +17,5 @@
   <xacro:include filename="$(find ros_industrial_support)/urdf/computer_mobile/computer.urdf.xacro"/>
   <xacro:computer_urdf computer_parent="world" computer_prefix="comp_mobile_" >
-  <origin xyz="1.5 -0.5 0" rpy="0 0 ${radians(45)}"/>
+  <origin xyz="1.5 -0.5 0.00" rpy="0 0 ${radians(45)}"/>
   </xacro:computer_urdf>
   <!-- Robot1 Pedestal -->

File: 5_transferframes/transferframes_moveit_config/config/manipuation_environment.urdf.xacro (robot description, xacro)
@@ -3,5 +3,5 @@
     <xacro:arg name="initial_positions_file" default="initial_positions.yaml" />
     <!-- Import manipuation_environment urdf file -->
-    <xacro:include filename="$(find manipulation)/urdf/environment.urdf.xacro" />
+    <xacro:include filename="$(find transferframes)/urdf/environment.urdf.xacro" />
     <!-- Import control_xacro -->
     <xacro:include filename="manipuation_environment.ros2_control.xacro" />

File: support/ros_industrial_support/urdf/bin/bin.urdf.xacro (robot description, xacro)
@@ -3,5 +3,7 @@
   <xacro:arg name="mesh_path" default="$(find ros_industrial_support)"/>
   <!--<xacro:macro name="bin_urdf" params="prefix mesh_path:='package://ros_industrial_support'">-->
+  <!--<xacro:macro name="bin_urdf" params="prefix mesh_path:='$(find ros_industrial_support)'">-->
   <xacro:macro name="bin_urdf" params="prefix">
+  <xacro:property name="mesh_path" value="file://$(find ros_industrial_support)"/>
     <!-- link list -->
     <link name="${prefix}base_link">
@@ -9,6 +11,5 @@
         <origin xyz="0 0 0" rpy="0 0 0" />
         <geometry>
-          <mesh filename="$(find ros_industrial_support)/meshes/bin/visual/bin.dae" />
-          <mesh filename="package://ros_industrial_support/meshes/bin/visual/bin.dae" />
+          <mesh filename="${mesh_path}/meshes/bin/visual/bin.dae" />
           <scale>0.6 0.6 0.6</scale>
         </geometry>
@@ -17,5 +18,5 @@
         <origin xyz="0 0 0" rpy="0 0 0"/>
         <geometry>
-          <mesh filename="$(find ros_industrial_support)/meshes/bin/collision/bin_bottom.dae"/>
+          <mesh filename="${mesh_path}/meshes/bin/collision/bin_bottom.dae"/>
           <scale>0.6 0.6 0.6</scale>
         </geometry>
@@ -24,5 +25,5 @@
         <origin xyz="0 0 0" rpy="0 0 0"/>
         <geometry>
-          <mesh filename="$(find ros_industrial_support)/meshes/bin/collision/bin_sides.dae"/>
+          <mesh filename="${mesh_path}/meshes/bin/collision/bin_sides.dae"/>
           <scale>0.6 0.6 0.6</scale>
         </geometry>

File: support/ros_industrial_support/urdf/computer_mobile/computer.urdf.xacro (robot description, xacro)
@@ -1,5 +1,7 @@
 <?xml version="1.0" ?>
 <robot name="computer_urdf" xmlns:xacro="http://www.ros.org/wiki/xacro">
-    <xacro:macro name="computer_urdf" params="computer_parent computer_prefix mesh_path:='package://ros_industrial_support' *origin">
+  <!--<xacro:macro name="computer_urdf" params="computer_parent computer_prefix mesh_path:='package://ros_industrial_support' *origin">-->
+  <xacro:macro name="computer_urdf" params="computer_parent computer_prefix  *origin">
+  <xacro:property name="mesh_path" value="file://$(find ros_industrial_support)"/>
   <joint name="${computer_prefix}joint" type="fixed">
     <xacro:insert_block name="origin" />
@@ -26,7 +28,10 @@
                  iyy="1.0" iyz="0"
                  izz="1.0" />
-        <mass value="100" />
+        <mass value="1.0" />
       </inertial>
     </link>
+    <gazebo>
+      <static>true</static>
+    </gazebo>
   </xacro:macro>
 </robot>

File: support/ros_industrial_support/urdf/workcell/workcell.urdf.xacro (robot description, xacro)
@@ -25,5 +25,5 @@
       <parent link="${workcell_parent}" />
       <child link="workcell" />
-      <origin xyz="0 0 0" rpy="0 0 ${radians(90)}" />
+      <origin xyz="0 0 0.0" rpy="0 0 ${radians(90)}" />
     </joint>
   </xacro:macro>

Commit message: 20241201

File: 5_transferframes/transferframes/urdf/environment.urdf.xacro (robot description, xacro)
@@ -24,4 +24,8 @@
     <origin xyz="-0.0 0 0.0" rpy="0 0 0"/>
   </xacro:robot_pedestal_urdf>
+  <xacro:include filename="$(find ros_industrial_support)/urdf/logical_camera/logical_camera.urdf.xacro"/>
+  <xacro:logical_camera_urdf logical_camera_prefix="camera1_" logical_camera_parent="world">
+    <origin xyz="0.5 -0.5 2.0" rpy="0 0 0"/>
+  </xacro:logical_camera_urdf>
  <!-- Robot1 -->
   <xacro:include filename="$(find ros_industrial_support)/urdf/ufactory/ufactory_xarm6.urdf.xacro"/>

Commit message: 20251202-1

File: 5_transferframes/transferframes/urdf/environment.urdf.xacro (robot description, xacro)
@@ -59,3 +59,14 @@
     <child link="vacuum_gripper1_base_link" />
   </joint>
+    <plugin name="vacuum_gripper" filename="libgazebo_ros_vacuum_gripper.so">
+      <ros>
+        <namespace>/robot</namespace>
+        <remapping>
+          <remap from="~/grasp" to="/gripper/grasp"/>
+        </remapping>
+      </ros>
+      <link_name>link_eef</link_name>
+      <!-- Max distance to attract entities -->
+      <max_distance>10.0</max_distance>
+    </plugin>
 </robot>

File: support/ros_industrial_support/urdf/ufactory/ufactory_xarm6.urdf.xacro (robot description, xacro)
@@ -64,5 +64,5 @@
   <link name="${prefix}base_link"/>
   <link name="${prefix}tool_link"/>
-  <joint name="${prefix}tool_link" type="fixed">
+  <joint name="${prefix}eff_to_tool" type="fixed">
     <origin xyz="0 0 0" rpy="0 0 0" />
     <parent link="${prefix}link_eef" />

File: support/ros_industrial_support/urdf/vacuum_gripper/vacuum_gripper.urdf.xacro (robot description, xacro)
@@ -28,32 +28,8 @@
       </inertial>
     </link>
-    <link name="${prefix}suction_cup">
-      <visual>
-        <origin xyz="0 0 0" rpy="0 0 0" />
-        <geometry>
-          <box size="0.001 0.001 0.001" />
-        </geometry>
-        <material name="red">
-          <color rgba="1 0 0 1"/>
-        </material>
-      </visual>
-      <collision>
-        <origin xyz="0 0 0" rpy="0 0 0"/>
-        <geometry>
-          <box size="0.001 0.001 0.001" />
-        </geometry>
-        <material name="red"/>
-      </collision>
-      <inertial>
-        <origin xyz="0 0 0" rpy="0 0 0" />
-        <inertia ixx="0.0001" ixy="0" ixz="0"
-                 iyy="0.0001" iyz="0"
-                 izz="0.0001" />
-        <mass value="0.00001" />
-      </inertial>
-    </link>
+    <link name="${prefix}suction_cup"/>
     <!-- joint list -->
     <joint name="${joint_prefix}" type="fixed">
-      <origin xyz="0 0 0.01" rpy="0 0 0" />
+      <origin xyz="0 0 0.08" rpy="0 0 0" />
       <parent link="${prefix}base_link" />
       <child link="${prefix}suction_cup" />

Commit message: 20241203-1

File: 5_transferframes/transferframes/urdf/environment.urdf.xacro (robot description, xacro)
@@ -24,11 +24,10 @@
     <origin xyz="-0.0 0 0.0" rpy="0 0 0"/>
   </xacro:robot_pedestal_urdf>
-  <!--
+  <!-- Camera1 -->
   <xacro:include filename="$(find ros_industrial_support)/urdf/logical_camera/logical_camera.urdf.xacro"/>
   <xacro:logical_camera_urdf logical_camera_prefix="camera1_" logical_camera_parent="world">
-    <origin xyz="0.5 -0.5 2.0" rpy="0 0 0"/>
+    <origin xyz="0.5 -0.7 2.0" rpy="0 ${radians(90)} 0"/>
   </xacro:logical_camera_urdf>
-  -->
- <!-- Robot1 -->
+  <!-- Robot1 -->
   <xacro:include filename="$(find ros_industrial_support)/urdf/ufactory/ufactory_xarm6.urdf.xacro"/>
   <xacro:ufactory_xarm6 prefix="" joint_limited="true"/>
@@ -38,7 +37,4 @@
   <!-- bins -->
   <xacro:include filename="$(find ros_industrial_support)/urdf/bin/bin.urdf.xacro"/>
-  <!--
-  <xacro:bin_urdf prefix="bin_1_" mesh_path="package://ros_industrial_support"/>
-  -->
   <xacro:bin_urdf prefix="bin_1_"/>
   <!-- bin to world. -->
@@ -59,14 +55,3 @@
     <child link="vacuum_gripper1_base_link" />
   </joint>
-    <plugin name="vacuum_gripper" filename="libgazebo_ros_vacuum_gripper.so">
-      <ros>
-        <namespace>/robot</namespace>
-        <remapping>
-          <remap from="~/grasp" to="/gripper/grasp"/>
-        </remapping>
-      </ros>
-      <link_name>link_eef</link_name>
-      <!-- Max distance to attract entities -->
-      <max_distance>10.0</max_distance>
-    </plugin>
 </robot>

File: support/ros_industrial_support/urdf/assembly_station/assembly_station.urdf.xacro (robot description, xacro)
@@ -15,7 +15,4 @@
   </joint>
     <!-- Links -->
-<!--
-<link name="${assembly_station_parent}"/>
--->
     <link name="${assembly_station_prefix}origin">
       <visual>

File: support/ros_industrial_support/urdf/logical_camera/logical_camera.urdf.xacro (robot description, xacro)
@@ -1,41 +1,38 @@
-<?xml version="1.0"?>
+<?xml version="1.0" ?>
 <robot name="logical_camera_urdf" xmlns:xacro="http://www.ros.org/wiki/xacro">
-  <xacro:macro name="logical_camera_urdf" params="logical_camera_prefix logical_camera_parent *origin">
-    <xacro:property name="length" value="0.2"/>
-    <xacro:property name="width" value="0.050"/>
-    <xacro:property name="height" value="0.050"/>
-    <joint name="${logical_camera_prefix}logical_camera_joint" type="fixed">
-      <xacro:insert_block name="origin" />
-      <parent link="${logical_camera_parent}"/>
-      <child link="${logical_camera_prefix}base_link"/>
-    </joint>
-    <!-- link list -->
-    <link name="${logical_camera_prefix}base_link">
+  <xacro:macro name="logical_camera_urdf" params="logical_camera_parent logical_camera_prefix  *origin">
+  <xacro:property name="mesh_path" value="file://$(find ros_industrial_support)"/>
+  <joint name="${logical_camera_prefix}joint" type="fixed">
+    <xacro:insert_block name="origin" />
+    <parent link="${logical_camera_parent}"/>
+    <child link="${logical_camera_prefix}origin"/>
+  </joint>
+  <link name="${logical_camera_prefix}origin"/>
+  <joint name="${logical_camera_prefix}joint_post" type="fixed">
+    <origin xyz="-0.02 0 -0.02" rpy="0 0 -1.5708"/>
+    <parent link="${logical_camera_prefix}origin"/>
+    <child link="${logical_camera_prefix}origin_post"/>
+  </joint>
+    <!-- Links -->
+    <link name="${logical_camera_prefix}origin_post">
       <visual>
-        <origin xyz="0 0 ${height / 2}" rpy="0 0 0" />
         <geometry>
-          <box size="${width} ${length} ${height}" />
+          <mesh filename="${mesh_path}/meshes/camera/visual/camera.dae"/>
         </geometry>
-        <material name="dark_grey">
-          <color rgba="0.1 1.0 0.1 1.0"/>
-        </material>
       </visual>
       <collision>
-        <origin xyz="0 0 ${height / 2}" rpy="0 0 0" />
         <geometry>
-          <box size="${width} ${length} ${height}" />
+          <mesh filename="${mesh_path}/meshes/camera/collision/camera.dae"/>
         </geometry>
-        <material name="dark_grey"/>
       </collision>
       <inertial>
-        <origin xyz="0 0 0" rpy="0 0 0" />
-        <inertia ixx="0.1" ixy="0" ixz="0"
-                 iyy="0.1" iyz="0"
-                 izz="0.1" />
-        <mass value="1" />
+        <inertia ixx="1.0" ixy="0" ixz="0"
+                 iyy="1.0" iyz="0"
+                 izz="1.0" />
+        <mass value="1.0" />
       </inertial>
     </link>
-    <gazebo reference="${logical_camera_prefix}base_link">
-      <material>Gazebo/Green</material>
+    <gazebo>
+      <static>true</static>
     </gazebo>
   </xacro:macro>

File: support/ros_industrial_support/urdf/vacuum_gripper/vacuum_gripper.urdf.xacro (robot description, xacro)
@@ -36,4 +36,5 @@
       <child link="${prefix}suction_cup" />
     </joint>
+    <!--
     <gazebo>
       <plugin name="vacuum_gripper" filename="libgazebo_ros_vacuum_gripper.so">
@@ -45,8 +46,11 @@
           </ros>
           <link_name>"${prefix}suction_cup"</link_name>
+    -->
           <!-- Max distance to attract entities -->
+    <!--
           <max_distance>10.0</max_distance>
       </plugin>
     </gazebo>
+    -->
   </xacro:macro>
 </robot>
