Commit message: 20241213

File: 5_transferframes/transferframes/urdf/tmp.urdf (robot description, URDF)
Before this commit: robot manipuation_environment, 21 links, 20 joints
Links:
- link link1: geometry collision mesh filename=file:///home/student/xarm_ws/install/xarm_description/share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; visual mesh filename=file:///home/student/xarm_ws/install/xarm_description/share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
- link link2: geometry collision mesh filename=file:///home/student/xarm_ws/install/xarm_description/share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; visual mesh filename=file:///home/student/xarm_ws/install/xarm_description/share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
- link link3: geometry collision mesh filename=file:///home/student/xarm_ws/install/xarm_description/share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; visual mesh filename=file:///home/student/xarm_ws/install/xarm_description/share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
- link link4: geometry collision mesh filename=file:///home/student/xarm_ws/install/xarm_description/share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; visual mesh filename=file:///home/student/xarm_ws/install/xarm_description/share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
- link link5: geometry collision mesh filename=file:///home/student/xarm_ws/install/xarm_description/share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; visual mesh filename=file:///home/student/xarm_ws/install/xarm_description/share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
- link link6: geometry collision mesh filename=file:///home/student/xarm_ws/install/xarm_description/share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; visual mesh filename=file:///home/student/xarm_ws/install/xarm_description/share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
- link link_base: geometry collision mesh filename=file:///home/student/xarm_ws/install/xarm_description/share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; visual mesh filename=file:///home/student/xarm_ws/install/xarm_description/share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
- link vacuum_gripper1_base_link: mass 1.0 -> 0.01; geometry collision cylinder length=0.01 radius=0.05; visual mesh filename=file:///home/student/ros2_industrial_ws/install/ros_industr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
- link vacuum_gripper1_suction_cup: mass None -> 0.001; geometry collision box size=0.001 0.001 0.001; visual box size=0.001 0.001 0.001

File: support/ros_industrial_support/urdf/ufactory/ufactory_xarm6.urdf.xacro (robot description, xacro)
@@ -69,4 +69,14 @@
     <child link="${prefix}tool_link" />
   </joint>
+  <!-- dit werkt ook niet -->
+  <gazebo reference="${prefix}base_link">
+      <material>Gazebo/Black</material>
+  </gazebo>
+  <gazebo reference="${prefix}tool_link">
+      <material>Gazebo/Black</material>
+  </gazebo>
+  <gazebo reference="${prefix}link_eef">
+      <material>Gazebo/Black</material>
+  </gazebo>
   </xacro:macro>
 </robot>

File: support/ros_industrial_support/urdf/vacuum_gripper/vacuum_gripper.urdf.xacro (robot description, xacro)
@@ -14,5 +14,6 @@
         </material>
       </visual>
-      <collision>
+      <collision name="${prefix}base_link_collision">
+        <!--
         <origin xyz="0 0 0" rpy="0 0 0"/>
         <geometry>
@@ -20,5 +21,11 @@
         </geometry>
         <material name="red"/>
+        -->
+        <geometry>
+          <!-- <mesh filename="file://$(find ariac_description)/meshes/vacuum_gripper/vacuum_gripper.stl" scale="1 1 1"/> -->
+          <cylinder radius="0.05" length="0.01" />
+        </geometry>
       </collision>
+      <!--
       <inertial>
         <origin xyz="0 0 0" rpy="0 0 0" />
@@ -27,4 +34,10 @@
                  izz="1.0" />
         <mass value="1.0" />
+      </inertial>
+      -->
+      <inertial>
+        <origin xyz="0 0 0" rpy="0 0 0"/>
+        <mass value="0.01"/>
+        <inertia ixx="0.0000063" ixy="0.0" ixz="0.0" iyy="0.0000063" iyz="0.0" izz="0.000025"/>
       </inertial>
     </link>
@@ -64,4 +77,7 @@
       </sensor>
     </gazebo>
+    <gazebo reference="${prefix}base_link">
+      <material>Gazebo/Green</material>
+    </gazebo>
     <gazebo reference="vacuum_gripper1_suction_cup">
       <material>Gazebo/Black</material>
@@ -76,6 +92,5 @@
             <remapping>grasping:=custom_grasping</remapping>
           </ros>
-        <!--<link_name>${prefix}suction_cup</link_name>-->
-        <link_name>xarm:link6</link_name>
+        <link_name>${prefix}suction_cup</link_name>
         <!--<link_name>vacuum_gripper1_suction_cup</link_name>-->
         <!-- Max distance to attract entities -->

Commit message: 20241215

File: 5_transferframes/transferframes/urdf/tmp.urdf (robot description, URDF)
Before this commit: robot manipuation_environment, 21 links, 20 joints
Links:
- link assembly_station_origin: geometry collision mesh filename=file:///home/gerard/ros_industrial_ws/install/ros_industria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 scale=1.1 1.1 1.1; visual mesh filename=file:///home/gerard/ros_industrial_ws/install/ros_industria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 scale=1.1 1.1 1.1
- link bin_1_base_link: geometry collision mesh filename=file:///home/gerard/ros_industrial_ws/install/ros_industria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; collision mesh filename=file:///home/gerard/ros_industrial_ws/install/ros_industria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
- link camera1_origin_post: geometry collision mesh filename=file:///home/gerard/ros_industrial_ws/install/ros_industria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; visual mesh filename=file:///home/gerard/ros_industrial_ws/install/ros_industria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
- link comp_mobile_origin: geometry collision mesh filename=file:///home/gerard/ros_industrial_ws/install/ros_industria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 scale=0.01 0.01 0.01; visual mesh filename=file:///home/gerard/ros_industrial_ws/install/ros_industria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 scale=0.01 0.01 0.01
- link link1: geometry collision mesh filename=file:///home/gerard/ros_industrial_ws/install/xarm_descript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; visual mesh filename=file:///home/gerard/ros_industrial_ws/install/xarm_descript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
- link link2: geometry collision mesh filename=file:///home/gerard/ros_industrial_ws/install/xarm_descript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; visual mesh filename=file:///home/gerard/ros_industrial_ws/install/xarm_descript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
- link link3: geometry collision mesh filename=file:///home/gerard/ros_industrial_ws/install/xarm_descript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; visual mesh filename=file:///home/gerard/ros_industrial_ws/install/xarm_descript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
- link link4: geometry collision mesh filename=file:///home/gerard/ros_industrial_ws/install/xarm_descript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; visual mesh filename=file:///home/gerard/ros_industrial_ws/install/xarm_descript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
- link link5: geometry collision mesh filename=file:///home/gerard/ros_industrial_ws/install/xarm_descript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; visual mesh filename=file:///home/gerard/ros_industrial_ws/install/xarm_descript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
- link link6: geometry collision mesh filename=file:///home/gerard/ros_industrial_ws/install/xarm_descript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; visual mesh filename=file:///home/gerard/ros_industrial_ws/install/xarm_descript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
- link link_base: geometry collision mesh filename=file:///home/gerard/ros_industrial_ws/install/xarm_descript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; visual mesh filename=file:///home/gerard/ros_industrial_ws/install/xarm_descript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
- link vacuum_gripper1_base_link: geometry collision cylinder length=0.01 radius=0.05; visual mesh filename=file:///home/gerard/ros_industrial_ws/install/ros_industria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
