Commit message: 20241203

File: support/ros_industrial_support/urdf/vacuum_gripper/vacuum_gripper.urdf.xacro (robot description, xacro)
@@ -2,4 +2,5 @@
 <robot xmlns:xacro="http://www.ros.org/wiki/xacro">
   <xacro:macro name="vacuum_gripper_urdf" params="prefix joint_prefix">
+  <xacro:property name="mesh_path" value="file://$(find ros_industrial_support)"/>
     <!-- link list -->
     <link name="${prefix}base_link">
@@ -7,5 +8,5 @@
         <origin xyz="0 0 0" rpy="0 0 0" />
         <geometry>
-          <mesh filename="package://ros_industrial_support/meshes/vacuum_gripper/visual/vacuum_gripper.dae"/>
+          <mesh filename="${mesh_path}/meshes/vacuum_gripper/visual/vacuum_gripper.dae"/>
         </geometry>
         <material name="red">
@@ -16,5 +17,5 @@
         <origin xyz="0 0 0" rpy="0 0 0"/>
         <geometry>
-          <mesh filename="package://ros_industrial_support/meshes/vacuum_gripper/collision/vacuum_gripper.dae"/>
+          <mesh filename="${mesh_path}/meshes/vacuum_gripper/collision/vacuum_gripper.dae"/>
         </geometry>
         <material name="red"/>
@@ -35,4 +36,17 @@
       <child link="${prefix}suction_cup" />
     </joint>
+    <gazebo>
+      <plugin name="vacuum_gripper" filename="libgazebo_ros_vacuum_gripper.so">
+          <ros>
+              <namespace>/robot</namespace>
+              <remapping>
+                  <remap from="~/grasp" to="/gripper/grasp"/>
+              </remapping>
+          </ros>
+          <link_name>"${prefix}suction_cup"</link_name>
+          <!-- Max distance to attract entities -->
+          <max_distance>10.0</max_distance>
+      </plugin>
+    </gazebo>
   </xacro:macro>
 </robot>

File: support/ros_industrial_support/urdf/workcell/workcell.urdf.xacro (robot description, xacro)
@@ -2,4 +2,5 @@
 <robot name="workcell_urdf" xmlns:xacro="http://www.ros.org/wiki/xacro">
     <xacro:macro name="workcell_urdf" params="workcell_parent">
+    <xacro:property name="mesh_path" value="file://$(find ros_industrial_support)"/>
     <!-- Links -->
     <link name="world_interface"/>
@@ -7,10 +8,10 @@
       <visual>
         <geometry>
-          <mesh filename="package://ros_industrial_support/meshes/workcell/visual/workcell.dae"/>
+          <mesh filename="${mesh_path}/meshes/workcell/visual/workcell.dae"/>
         </geometry>
       </visual>
       <collision>
         <geometry>
-          <mesh filename="package://ros_industrial_support/meshes/workcell/collision/workcell.dae"/>
+          <mesh filename="${mesh_path}/meshes/workcell/collision/workcell.dae"/>
         </geometry>
       </collision>

Commit message: 20241220

File: support/ros_industrial_support/urdf/vacuum_gripper/vacuum_gripper.urdf.xacro (robot description, xacro)
@@ -24,5 +24,5 @@
         <geometry>
           <!-- <mesh filename="file://$(find ariac_description)/meshes/vacuum_gripper/vacuum_gripper.stl" scale="1 1 1"/> -->
-          <cylinder radius="0.05" length="0.01" />
+          <cylinder radius="0.045" length="0.01" />
         </geometry>
       </collision>
@@ -96,5 +96,4 @@
         <!--<link_name>vacuum_gripper1_suction_cup</link_name>-->
         <!-- Max distance to attract entities -->
-        <max_distance>55.0</max_distance>
       </plugin>
     </gazebo>

Commit message: 20241222

File: support/ros_industrial_support/urdf/vacuum_gripper/vacuum_gripper.urdf.xacro (robot description, xacro)
@@ -15,25 +15,8 @@
       </visual>
       <collision name="${prefix}base_link_collision">
-        <!--
-        <origin xyz="0 0 0" rpy="0 0 0"/>
         <geometry>
           <mesh filename="${mesh_path}/meshes/vacuum_gripper/collision/vacuum_gripper.dae"/>
         </geometry>
-        <material name="red"/>
-        -->
-        <geometry>
-          <!-- <mesh filename="file://$(find ariac_description)/meshes/vacuum_gripper/vacuum_gripper.stl" scale="1 1 1"/> -->
-          <cylinder radius="0.045" length="0.01" />
-        </geometry>
       </collision>
-      <!--
-      <inertial>
-        <origin xyz="0 0 0" rpy="0 0 0" />
-        <inertia ixx="1.0" ixy="0" ixz="0"
-                 iyy="1.0" iyz="0"
-                 izz="1.0" />
-        <mass value="1.0" />
-      </inertial>
-      -->
       <inertial>
         <origin xyz="0 0 0" rpy="0 0 0"/>
@@ -43,27 +26,8 @@
     </link>
     <link name="${prefix}suction_cup">
-      <visual>
-        <origin xyz="0 0 0"/>
-        <geometry>
-          <box size="0.001 0.001 0.001"/>
-        </geometry>
-      </visual>
-      <collision>
-        <origin xyz="0 0 0"/>
-        <geometry>
-          <box size="0.001 0.001 0.001"/>
-        </geometry>
-      </collision>
-      <inertial>
-        <origin xyz="0 0 0" rpy="0 0 0" />
-        <inertia ixx="0.001" ixy="0" ixz="0"
-                 iyy="0.001" iyz="0"
-                 izz="0.001" />
-        <mass value="0.001" />
-      </inertial>
     </link>
     <!-- joint list -->
     <joint name="${joint_prefix}" type="fixed">
-      <origin xyz="0 0 0.08" rpy="0 0 0" />
+      <origin xyz="0 0 0.080" rpy="0 0 0" />
       <parent link="${prefix}base_link" />
       <child link="${prefix}suction_cup" />
@@ -84,16 +48,12 @@
     </gazebo>
     <gazebo>
-      <!--<plugin name="vacuum_gripper" filename="libgazebo_ros_vacuum_gripper.so">-->
-      <plugin filename="libMyVacuumGripperPlugin.so" name="vacuum_gripper">
+      <plugin filename="libCustomVacuumGripperPlugin.so" name="vacuum_gripper">
           <ros>
             <!--<namespace>/gazebo_plugins</namespace>-->
-            <namespace>/ros_industrial_actuators</namespace>
+            <namespace>/gripper</namespace>
             <remapping>switch:=custom_switch</remapping>
             <remapping>grasping:=custom_grasping</remapping>
           </ros>
-        <!--<link_name>xarm::${prefix}suction_cup</link_name>-->
         <link_name>xarm::link6</link_name>
-        <!--<link_name>vacuum_gripper1_suction_cup</link_name>-->
-        <!-- Max distance to attract entities -->
       </plugin>
     </gazebo>
