Commit message: 20261209

File: tmp.urdf (robot description, URDF)
Before this commit: robot robot, 3 links, 2 joints
Links:
- link workcell: geometry collision mesh filename=file:///home/student/ros2_industrial_ws/install/ros_industr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; visual mesh filename=file:///home/student/ros2_industrial_ws/install/ros_industr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
