Commit message: 20241201

File: support/ros_industrial_support/urdf/computer_mobile/computer.urdf.xacro (robot description, xacro)
@@ -1,5 +1,4 @@
 <?xml version="1.0" ?>
 <robot name="computer_urdf" xmlns:xacro="http://www.ros.org/wiki/xacro">
-  <!--<xacro:macro name="computer_urdf" params="computer_parent computer_prefix mesh_path:='package://ros_industrial_support' *origin">-->
   <xacro:macro name="computer_urdf" params="computer_parent computer_prefix  *origin">
   <xacro:property name="mesh_path" value="file://$(find ros_industrial_support)"/>

Commit message: 20250423-2

File: support/ros_industrial_support/urdf/computer_mobile/computer.urdf.xacro (robot description, xacro)
@@ -2,5 +2,5 @@
 <robot name="computer_urdf" xmlns:xacro="http://www.ros.org/wiki/xacro">
   <xacro:macro name="computer_urdf" params="computer_parent computer_prefix  *origin">
-  <xacro:property name="mesh_path" value="file://$(find ros_industrial_support)"/>
+  <xacro:property name="mesh_path" value="file://$(find ros_industrial_gazebo)"/>
   <joint name="${computer_prefix}joint" type="fixed">
     <xacro:insert_block name="origin" />
@@ -15,10 +15,10 @@
       <visual>
         <geometry>
-          <mesh filename="${mesh_path}/meshes/computer_mobile/meshes/computer.dae" scale="0.01 0.01 0.01"/>
+          <mesh filename="${mesh_path}/models/computer_mobile/meshes/computer.dae" scale="0.01 0.01 0.01"/>
         </geometry>
       </visual>
       <collision>
         <geometry>
-          <mesh filename="${mesh_path}/meshes/computer_mobile/meshes/computer.dae" scale="0.01 0.01 0.01"/>
+          <mesh filename="${mesh_path}/models/computer_mobile/meshes/computer.dae" scale="0.01 0.01 0.01"/>
         </geometry>
       </collision>
