Commit message: 20250506

File: 4_manipulation/manipulation/urdf/robot_on_pedestal.urdf.xacro (robot description, xacro)
@@ -3,20 +3,4 @@
   <!-- world -->
   <link name="world" />
-  <!-- hall -->
-  <!--
-  <xacro:include filename="$(find ros_industrial_support)/urdf/hall/hall.urdf.xacro"/>
-  <xacro:hall_urdf hall_prefix="hall_" hall_parent="world">
-    <origin xyz="-2.5 0 0.0" rpy="0 0 0"/>
-  </xacro:hall_urdf>
-  -->
-  <xacro:include filename="$(find ros_industrial_support)/urdf/assembly_station/assembly_station.urdf.xacro"/>
-  <xacro:assembly_station_urdf assembly_station_prefix="assembly_station_" assembly_station_parent="world">
-    <origin xyz="0.5 -0.5 0.0" rpy="0 0 ${radians(90)}"/>
-  </xacro:assembly_station_urdf>
-  <!-- Mobile Computer -->
-  <xacro:include filename="$(find ros_industrial_support)/urdf/computer_mobile/computer.urdf.xacro"/>
-  <xacro:computer_urdf computer_parent="world" computer_prefix="comp_mobile_" >
-    <origin xyz="1.5 -0.5 0.05" rpy="0 0 ${radians(45)}"/>
-  </xacro:computer_urdf>
   <!-- Robot1 Pedestal -->
   <xacro:include filename="$(find ros_industrial_support)/urdf/robot_pedestal/robot_pedestal.urdf.xacro"/>
@@ -30,13 +14,4 @@
   <xacro:include filename="$(find ros_industrial_support)/urdf/vacuum_gripper/vacuum_gripper.urdf.xacro"/>
   <xacro:vacuum_gripper_urdf prefix="vacuum_gripper1_" joint_prefix="vacuum_gripper1_joint"/>
-  <!-- bins -->
-  <xacro:include filename="$(find ros_industrial_support)/urdf/bin/bin.urdf.xacro"/>
-  <xacro:bin_urdf prefix="bin_1_"/>
-  <!-- bin to world. -->
-  <joint name="bin_1_joint" type="fixed">
-    <parent link="world" />
-    <child link="bin_1_base_link" />
-    <origin xyz="-0.5 0.5 0.0" rpy="0 0 0" />
-  </joint>
   <!-- robot1 to pedestal. -->
   <joint name="robot1_to_pedestal" type="fixed">
