Commit message: 20241223

File: 4_manipulation/manipulation/urdf/environment.urdf.xacro (robot description, xacro)
@@ -11,5 +11,5 @@
   -->
   <xacro:include filename="$(find ros_industrial_support)/urdf/assembly_station/assembly_station.urdf.xacro"/>
-  <xacro:assembly_station_urdf assembly_station_prefix="shelf_" assembly_station_parent="world">
+  <xacro:assembly_station_urdf assembly_station_prefix="assembly_station_" assembly_station_parent="world">
     <origin xyz="0.5 -0.5 0.0" rpy="0 0 ${radians(90)}"/>
   </xacro:assembly_station_urdf>
@@ -17,5 +17,5 @@
   <xacro:include filename="$(find ros_industrial_support)/urdf/computer_mobile/computer.urdf.xacro"/>
   <xacro:computer_urdf computer_parent="world" computer_prefix="comp_mobile_" >
-  <origin xyz="1.5 -0.5 0" rpy="0 0 ${radians(45)}"/>
+  <origin xyz="1.5 -0.5 0.00" rpy="0 0 ${radians(45)}"/>
   </xacro:computer_urdf>
   <!-- Robot1 Pedestal -->
@@ -24,5 +24,5 @@
     <origin xyz="-0.0 0 0.0" rpy="0 0 0"/>
   </xacro:robot_pedestal_urdf>
- <!-- Robot1 -->
+  <!-- Robot1 -->
   <xacro:include filename="$(find ros_industrial_support)/urdf/ufactory/ufactory_xarm6.urdf.xacro"/>
   <xacro:ufactory_xarm6 prefix="" joint_limited="true"/>

Commit message: 20250328

File: 4_manipulation/manipulation/urdf/environment.urdf.xacro (robot description, xacro)
@@ -10,13 +10,17 @@
   </xacro:hall_urdf>
   -->
+<!--
   <xacro:include filename="$(find ros_industrial_support)/urdf/assembly_station/assembly_station.urdf.xacro"/>
   <xacro:assembly_station_urdf assembly_station_prefix="assembly_station_" assembly_station_parent="world">
     <origin xyz="0.5 -0.5 0.0" rpy="0 0 ${radians(90)}"/>
   </xacro:assembly_station_urdf>
+-->
   <!-- Mobile Computer -->
+  <!--
   <xacro:include filename="$(find ros_industrial_support)/urdf/computer_mobile/computer.urdf.xacro"/>
   <xacro:computer_urdf computer_parent="world" computer_prefix="comp_mobile_" >
   <origin xyz="1.5 -0.5 0.00" rpy="0 0 ${radians(45)}"/>
   </xacro:computer_urdf>
+  -->
   <!-- Robot1 Pedestal -->
   <xacro:include filename="$(find ros_industrial_support)/urdf/robot_pedestal/robot_pedestal.urdf.xacro"/>
@@ -31,7 +35,10 @@
   <xacro:vacuum_gripper_urdf prefix="vacuum_gripper1_" joint_prefix="vacuum_gripper1_joint"/>
   <!-- bins -->
+  <!--
   <xacro:include filename="$(find ros_industrial_support)/urdf/bin/bin.urdf.xacro"/>
   <xacro:bin_urdf prefix="bin_1_"/>
+  -->
   <!-- bin to world. -->
+  <!--
   <joint name="bin_1_joint" type="fixed">
     <parent link="world" />
@@ -39,8 +46,13 @@
     <origin xyz="-0.5 0.5 0.0" rpy="0 0 0" />
   </joint>
+  -->
   <!-- robot1 to pedestal. -->
   <joint name="robot1_to_pedestal" type="fixed">
     <origin xyz="0 0 1.15" rpy="0 0 ${radians(0)}" />
     <parent link="robot1_pedestal_link" />
+    <!--
+    <origin xyz="0 0 0.1" rpy="0 0 ${radians(0)}" />
+    <parent link="world" />
+    -->
     <child link="base_link" />
   </joint>

Commit message: 20250404

File: 4_manipulation/manipulation/urdf/environment.urdf.xacro (robot description, xacro)
@@ -10,15 +10,13 @@
   </xacro:hall_urdf>
   -->
-<!--
   <xacro:include filename="$(find ros_industrial_support)/urdf/assembly_station/assembly_station.urdf.xacro"/>
   <xacro:assembly_station_urdf assembly_station_prefix="assembly_station_" assembly_station_parent="world">
     <origin xyz="0.5 -0.5 0.0" rpy="0 0 ${radians(90)}"/>
   </xacro:assembly_station_urdf>
--->
   <!-- Mobile Computer -->
   <!--
   <xacro:include filename="$(find ros_industrial_support)/urdf/computer_mobile/computer.urdf.xacro"/>
   <xacro:computer_urdf computer_parent="world" computer_prefix="comp_mobile_" >
-  <origin xyz="1.5 -0.5 0.00" rpy="0 0 ${radians(45)}"/>
+    <origin xyz="1.5 -0.5 0.00" rpy="0 0 ${radians(45)}"/>
   </xacro:computer_urdf>
   -->

Commit message: 20250404-1

File: 4_manipulation/manipulation/urdf/environment.urdf.xacro (robot description, xacro)
@@ -33,10 +33,7 @@
   <xacro:vacuum_gripper_urdf prefix="vacuum_gripper1_" joint_prefix="vacuum_gripper1_joint"/>
   <!-- bins -->
-  <!--
   <xacro:include filename="$(find ros_industrial_support)/urdf/bin/bin.urdf.xacro"/>
   <xacro:bin_urdf prefix="bin_1_"/>
-  -->
   <!-- bin to world. -->
-  <!--
   <joint name="bin_1_joint" type="fixed">
     <parent link="world" />
@@ -44,13 +41,8 @@
     <origin xyz="-0.5 0.5 0.0" rpy="0 0 0" />
   </joint>
-  -->
   <!-- robot1 to pedestal. -->
   <joint name="robot1_to_pedestal" type="fixed">
     <origin xyz="0 0 1.15" rpy="0 0 ${radians(0)}" />
     <parent link="robot1_pedestal_link" />
-    <!--
-    <origin xyz="0 0 0.1" rpy="0 0 ${radians(0)}" />
-    <parent link="world" />
-    -->
     <child link="base_link" />
   </joint>

Commit message: 20250423

File: 4_manipulation/manipulation/urdf/environment.urdf.xacro (robot description, xacro)
@@ -15,10 +15,10 @@
   </xacro:assembly_station_urdf>
   <!-- Mobile Computer -->
-  <!--
+<!--
   <xacro:include filename="$(find ros_industrial_support)/urdf/computer_mobile/computer.urdf.xacro"/>
   <xacro:computer_urdf computer_parent="world" computer_prefix="comp_mobile_" >
     <origin xyz="1.5 -0.5 0.00" rpy="0 0 ${radians(45)}"/>
   </xacro:computer_urdf>
-  -->
+-->
   <!-- Robot1 Pedestal -->
   <xacro:include filename="$(find ros_industrial_support)/urdf/robot_pedestal/robot_pedestal.urdf.xacro"/>

File: 4_manipulation/manipulation_moveit_config/config/manipuation_environment.ros2_control.xacro (robot description, xacro)
@@ -2,5 +2,5 @@
 <robot xmlns:xacro="http://www.ros.org/wiki/xacro">
     <xacro:macro name="manipuation_environment_ros2_control" params="name initial_positions_file">
-        <xacro:property name="initial_positions" value="${xacro.load_yaml(initial_positions_file)['initial_positions']}"/>
+        <xacro:property name="initial_positions" value="${load_yaml(initial_positions_file)['initial_positions']}"/>
         <ros2_control name="${name}" type="system">
             <hardware>

Commit message: 20250507

File: 4_manipulation/manipulation/urdf/environment.urdf.xacro (robot description, xacro)
@@ -31,5 +31,5 @@
   <xacro:vacuum_gripper_urdf prefix="vacuum_gripper1_" joint_prefix="vacuum_gripper1_joint"/>
   <!-- bins -->
-  <xacro:include filename="$(find ros_industrial_support)/urdf/bin/bin.urdf.xacro"/>
+  <xacro:include filename="$(find ros_industrial_support)/urdf/drop_bin/drop_bin.urdf.xacro"/>
   <xacro:bin_urdf prefix="bin_1_"/>
   <!-- bin to world. -->

File: support/ros_industrial_support/urdf/assembly_station/assembly_station.urdf.xacro (robot description, xacro)
@@ -2,5 +2,5 @@
 <robot name="assembly_station_urdf" xmlns:xacro="http://www.ros.org/wiki/xacro">
     <xacro:macro name="assembly_station_urdf" params="assembly_station_parent assembly_station_prefix  *origin">
-    <xacro:property name="mesh_path" value="file://$(find ros_industrial_support)"/>
+  <xacro:property name="mesh_path" value="file://$(find ros_industrial_gazebo)"/>
   <joint name="${assembly_station_prefix}joint" type="fixed">
     <xacro:insert_block name="origin" />
@@ -18,10 +18,10 @@
       <visual>
         <geometry>
-          <mesh filename="${mesh_path}/meshes/assembly_station/meshes/assembly_station.dae" scale="1.1 1.1 1.1"/>
+          <mesh filename="${mesh_path}/models/assembly_station/meshes/assembly_station.dae" scale="1.1 1.1 1.1"/>
         </geometry>
       </visual>
       <collision>
         <geometry>
-          <mesh filename="${mesh_path}/meshes/assembly_station/meshes/assembly_station.dae" scale="1.1 1.1 1.1"/>
+          <mesh filename="${mesh_path}/models/assembly_station/meshes/assembly_station.dae" scale="1.1 1.1 1.1"/>
         </geometry>
       </collision>

File: support/ros_industrial_support/urdf/part_bin/part_bin.urdf.xacro (robot description, xacro)
@@ -5,5 +5,5 @@
   <!--<xacro:macro name="bin_urdf" params="prefix mesh_path:='$(find ros_industrial_support)'">-->
   <xacro:macro name="bin_urdf" params="prefix">
-  <xacro:property name="mesh_path" value="file://$(find ros_industrial_support)"/>
+  <xacro:property name="mesh_path" value="file://$(find ros_industrial_gazebo)"/>
     <!-- link list -->
     <link name="${prefix}base_link">
@@ -11,5 +11,12 @@
         <origin xyz="0 0 0" rpy="0 0 0" />
         <geometry>
-          <mesh filename="${mesh_path}/meshes/bin/visual/bin.dae" />
+          <mesh filename="${mesh_path}/models/part_bin/meshes/bin_exterior.dae" />
+          <scale>0.6 0.6 0.6</scale>
+        </geometry>
+      </visual>
+      <visual>
+        <origin xyz="0 0 0" rpy="0 0 0" />
+        <geometry>
+          <mesh filename="${mesh_path}/models/part_bin/meshes/bin_interior.stl" />
           <scale>0.6 0.6 0.6</scale>
         </geometry>
@@ -18,5 +25,5 @@
         <origin xyz="0 0 0" rpy="0 0 0"/>
         <geometry>
-          <mesh filename="${mesh_path}/meshes/bin/collision/bin_bottom.dae"/>
+          <mesh filename="${mesh_path}/models/part_bin/meshes/bin_exterior.dae"/>
           <scale>0.6 0.6 0.6</scale>
         </geometry>
@@ -25,5 +32,5 @@
         <origin xyz="0 0 0" rpy="0 0 0"/>
         <geometry>
-          <mesh filename="${mesh_path}/meshes/bin/collision/bin_sides.dae"/>
+          <mesh filename="${mesh_path}/models/part_bin/meshes/bin_interior.stl"/>
           <scale>0.6 0.6 0.6</scale>
         </geometry>
@@ -37,19 +44,4 @@
       </inertial>
     </link>
-    <link name="${prefix}drop_point">
-      <inertial>
-        <origin xyz="0 0 0" rpy="0 0 0" />
-        <inertia ixx="1.0" ixy="0" ixz="0"
-                 iyy="1.0" iyz="0"
-                 izz="1.0" />
-        <mass value="1.0" />
-      </inertial>
-    </link>
-    <!-- joint list -->
-    <joint name="${prefix}joint_1" type="fixed">
-      <origin xyz="0 0 1.0" rpy="0 0 0" />
-      <parent link="${prefix}base_link" />
-      <child link="${prefix}drop_point" />
-    </joint>
   </xacro:macro>
 </robot>
