Commit message: 20260227

File: 4_manipulation/manipulation/urdf/robot_on_pedestal.urdf (robot description, URDF)
Before this commit: robot manipuation_environment, 14 links, 13 joints
Links:
- link link1: geometry collision mesh filename=file:///home/gerard/xarm_ws/install/xarm_description/share/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; visual mesh filename=file:///home/gerard/xarm_ws/install/xarm_description/share/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
- link link2: geometry collision mesh filename=file:///home/gerard/xarm_ws/install/xarm_description/share/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; visual mesh filename=file:///home/gerard/xarm_ws/install/xarm_description/share/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
- link link3: geometry collision mesh filename=file:///home/gerard/xarm_ws/install/xarm_description/share/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; visual mesh filename=file:///home/gerard/xarm_ws/install/xarm_description/share/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
- link link4: geometry collision mesh filename=file:///home/gerard/xarm_ws/install/xarm_description/share/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; visual mesh filename=file:///home/gerard/xarm_ws/install/xarm_description/share/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
- link link5: geometry collision mesh filename=file:///home/gerard/xarm_ws/install/xarm_description/share/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; visual mesh filename=file:///home/gerard/xarm_ws/install/xarm_description/share/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
- link link6: geometry collision mesh filename=file:///home/gerard/xarm_ws/install/xarm_description/share/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; visual mesh filename=file:///home/gerard/xarm_ws/install/xarm_description/share/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
- link link_base: geometry collision mesh filename=file:///home/gerard/xarm_ws/install/xarm_description/share/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; visual mesh filename=file:///home/gerard/xarm_ws/install/xarm_description/share/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
- link vacuum_gripper1_base_link: geometry collision mesh filename=file:///home/gerard/ros2_industrial_ws/install/ros_industri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; visual mesh filename=file:///home/gerard/ros2_industrial_ws/install/ros_industri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
