Commit message: 20250106

File: 2_urdf/fanuc_robots/urdf/include/common_materials.xacro (robot description, xacro)
@@ -1,5 +1,5 @@
 <?xml version="1.0"?>
 <robot xmlns:xacro="http://wiki.ros.org/xacro">
-  <xacro:include filename="$(find urdf_basics)/urdf/include/common_colours.xacro"/>
+  <xacro:include filename="$(find fanuc_robots)/urdf/include/common_colours.xacro"/>
   <xacro:macro name="material_fanuc_yellow">
     <material name="">

File: 2_urdf/fanuc_robots/urdf/lrmate200ic.urdf.xacro (robot description, xacro)
@@ -1,5 +1,5 @@
 <?xml version="1.0" ?>
 <robot xmlns:xacro="http://wiki.ros.org/xacro">
-  <xacro:include filename="$(find urdf_basics)/urdf/include/common_materials.xacro"/>
+  <xacro:include filename="$(find fanuc_robots)/urdf/include/common_materials.xacro"/>
   <!-- NOTE: joint_limited is not used in this file -->
   <xacro:macro name="fanuc_lrmate200ic" params="prefix joint_limited:=false">
@@ -8,5 +8,5 @@
         <origin xyz="0 0 0" rpy="0 0 0"/>
         <geometry>
-          <mesh filename="package://urdf_basics/meshes/lrmate200ic/collision/base_link.stl"/>
+          <mesh filename="package://fanuc_robots/meshes/lrmate200ic/collision/base_link.stl"/>
         </geometry>
         <xacro:material_fanuc_gray24 />
@@ -15,5 +15,5 @@
         <origin xyz="0 0 0" rpy="0 0 0"/>
         <geometry>
-          <mesh filename="package://urdf_basics/meshes/lrmate200ic/collision/base_link.stl"/>
+          <mesh filename="package://fanuc_robots/meshes/lrmate200ic/collision/base_link.stl"/>
         </geometry>
       </collision>
@@ -23,5 +23,5 @@
         <origin xyz="0 0 0" rpy="0 0 0"/>
         <geometry>
-          <mesh filename="package://urdf_basics/meshes/lrmate200ic/collision/link_1.stl"/>
+          <mesh filename="package://fanuc_robots/meshes/lrmate200ic/collision/link_1.stl"/>
         </geometry>
         <xacro:material_fanuc_yellow />
@@ -30,5 +30,5 @@
         <origin xyz="0 0 0" rpy="0 0 0"/>
         <geometry>
-          <mesh filename="package://urdf_basics/meshes/lrmate200ic/collision/link_1.stl"/>
+          <mesh filename="package://fanuc_robots/meshes/lrmate200ic/collision/link_1.stl"/>
         </geometry>
       </collision>
@@ -38,5 +38,5 @@
         <origin xyz="0 0 0" rpy="0 0 0"/>
         <geometry>
-          <mesh filename="package://urdf_basics/meshes/lrmate200ic/collision/link_2.stl"/>
+          <mesh filename="package://fanuc_robots/meshes/lrmate200ic/collision/link_2.stl"/>
         </geometry>
         <xacro:material_fanuc_yellow />
@@ -45,5 +45,5 @@
         <origin xyz="0 0 0" rpy="0 0 0"/>
         <geometry>
-          <mesh filename="package://urdf_basics/meshes/lrmate200ic/collision/link_2.stl"/>
+          <mesh filename="package://fanuc_robots/meshes/lrmate200ic/collision/link_2.stl"/>
         </geometry>
       </collision>
@@ -53,5 +53,5 @@
         <origin xyz="0 0 0" rpy="0 0 0"/>
         <geometry>
-          <mesh filename="package://urdf_basics/meshes/lrmate200ic/collision/link_3.stl"/>
+          <mesh filename="package://fanuc_robots/meshes/lrmate200ic/collision/link_3.stl"/>
         </geometry>
         <xacro:material_fanuc_yellow />
@@ -60,5 +60,5 @@
         <origin xyz="0 0 0" rpy="0 0 0"/>
         <geometry>
-          <mesh filename="package://urdf_basics/meshes/lrmate200ic/collision/link_3.stl"/>
+          <mesh filename="package://fanuc_robots/meshes/lrmate200ic/collision/link_3.stl"/>
         </geometry>
       </collision>
@@ -68,5 +68,5 @@
         <origin xyz="0 0 0" rpy="0 0 0"/>
         <geometry>
-          <mesh filename="package://urdf_basics/meshes/lrmate200ic/collision/link_4.stl"/>
+          <mesh filename="package://fanuc_robots/meshes/lrmate200ic/collision/link_4.stl"/>
         </geometry>
         <xacro:material_fanuc_yellow />
@@ -75,5 +75,5 @@
         <origin xyz="0 0 0" rpy="0 0 0"/>
         <geometry>
-          <mesh filename="package://urdf_basics/meshes/lrmate200ic/collision/link_4.stl"/>
+          <mesh filename="package://fanuc_robots/meshes/lrmate200ic/collision/link_4.stl"/>
         </geometry>
       </collision>
@@ -83,5 +83,5 @@
         <origin xyz="0 0 0" rpy="0 0 0"/>
         <geometry>
-          <mesh filename="package://urdf_basics/meshes/lrmate200ic/collision/link_5.stl"/>
+          <mesh filename="package://fanuc_robots/meshes/lrmate200ic/collision/link_5.stl"/>
         </geometry>
         <xacro:material_fanuc_yellow />
@@ -90,5 +90,5 @@
         <origin xyz="0 0 0" rpy="0 0 0"/>
         <geometry>
-          <mesh filename="package://urdf_basics/meshes/lrmate200ic/collision/link_5.stl"/>
+          <mesh filename="package://fanuc_robots/meshes/lrmate200ic/collision/link_5.stl"/>
         </geometry>
       </collision>
@@ -98,5 +98,5 @@
         <origin xyz="0 0 0" rpy="0 0 0"/>
         <geometry>
-          <mesh filename="package://urdf_basics/meshes/lrmate200ic/collision/link_6.stl"/>
+          <mesh filename="package://fanuc_robots/meshes/lrmate200ic/collision/link_6.stl"/>
         </geometry>
         <xacro:material_fanuc_black />
@@ -105,5 +105,5 @@
         <origin xyz="0 0 0" rpy="0 0 0"/>
         <geometry>
-          <mesh filename="package://urdf_basics/meshes/lrmate200ic/collision/link_6.stl"/>
+          <mesh filename="package://fanuc_robots/meshes/lrmate200ic/collision/link_6.stl"/>
         </geometry>
       </collision>

File: 2_urdf/fanuc_robots/urdf/lrmate200ic_environment.urdf.xacro (robot description, xacro)
@@ -1,5 +1,5 @@
 <?xml version="1.0" ?>
 <robot name="fanuc_lrmate200ic" xmlns:xacro="http://wiki.ros.org/xacro">
-  <xacro:include filename="$(find urdf_basics)/urdf/robot/lrmate200ic.urdf.xacro"/>
+  <xacro:include filename="$(find fanuc_robots)/urdf/lrmate200ic.urdf.xacro"/>
   <xacro:fanuc_lrmate200ic prefix=""/>
 </robot>

File: 2_urdf/urdf_basics/urdf/assignment3.urdf.xacro (robot description, xacro)
@@ -72,9 +72,9 @@
   </joint>
   <!-- Update the below block for assignment 3 here -->
+  <xacro:include filename="$(find fanuc_robots)/urdf/lrmate200ic.urdf.xacro"/>
+  <xacro:fanuc_lrmate200ic prefix="robot2_"/>
   <!--
-  <xacro:include filename="$(find urdf_basics)/urdf/robot/lrmate200ic.urdf.xacro"/>
-  <xacro:fanuc_lrmate200ic prefix="robot2_"/>
+  <xacro:ufactory_xarm6 prefix="robot2_" joint_limited="true"/>
   -->
-  <xacro:ufactory_xarm6 prefix="robot2_" joint_limited="true"/>
   <!-- robot2 to pedestal. -->
   <joint name="robot2_to_pedestal" type="fixed">

Commit message: added urdf_demo

File: 2_urdf/fanuc_robots/urdf/include/common_materials.xacro (robot description, xacro)
@@ -3,70 +3,70 @@
   <xacro:include filename="$(find fanuc_robots)/urdf/include/common_colours.xacro"/>
   <xacro:macro name="material_fanuc_yellow">
-    <material name="">
+    <material name="fanuc_yellow">
       <color rgba="${color_fanuc_yellow}"/>
     </material>
   </xacro:macro>
   <xacro:macro name="material_fanuc_white">
-    <material name="">
+    <material name="fanuc_white">
       <color rgba="${color_fanuc_white}"/>
     </material>
   </xacro:macro>
   <xacro:macro name="material_fanuc_grey">
-    <material name="">
+    <material name="fanuc_grey">
       <color rgba="${color_fanuc_grey}"/>
     </material>
   </xacro:macro>
   <xacro:macro name="material_fanuc_gray24">
-    <material name="">
+    <material name="fanuc_gray24">
       <color rgba="${color_fanuc_gray24}"/>
     </material>
   </xacro:macro>
   <xacro:macro name="material_fanuc_gray28">
-    <material name="">
+    <material name="fanuc_gray28">
       <color rgba="${color_fanuc_gray28}"/>
     </material>
   </xacro:macro>
   <xacro:macro name="material_fanuc_gray31">
-    <material name="">
+    <material name="fanuc_gray31">
       <color rgba="${color_fanuc_gray31}"/>
     </material>
   </xacro:macro>
   <xacro:macro name="material_fanuc_gray40">
-    <material name="">
+    <material name="fanuc_gray40">
       <color rgba="${color_fanuc_gray40}"/>
     </material>
   </xacro:macro>
   <xacro:macro name="material_fanuc_yellow1">
-    <material name="">
+    <material name="fanuc_yellow1">
       <color rgba="${color_fanuc_yellow1}"/>
     </material>
   </xacro:macro>
   <xacro:macro name="material_fanuc_BAB0B0">
-    <material name="">
+    <material name="fanuc_BAB0B0">
       <color rgba="${color_fanuc_BAB0B0}"/>
     </material>
   </xacro:macro>
   <xacro:macro name="material_fanuc_E6E6E6">
-    <material name="">
+    <material name="fanuc_E6E6E6">
       <color rgba="${color_fanuc_E6E6E6}"/>
     </material>
   </xacro:macro>
   <xacro:macro name="material_fanuc_00FF73">
-    <material name="">
+    <material name="fanuc_00FF73">
       <color rgba="${color_fanuc_00FF73}"/>
     </material>
   </xacro:macro>
   <xacro:macro name="material_fanuc_black">
-    <material name="">
+    <material name="fanuc_black">
       <color rgba="${color_fanuc_black}"/>
     </material>
   </xacro:macro>
   <xacro:macro name="material_fanuc_greyish">
-    <material name="">
+    <material name="fanuc_greyish">
       <color rgba="${color_fanuc_greyish}"/>
     </material>
   </xacro:macro>
   <xacro:macro name="material_fanuc_green">
-    <material name="">
+    <material name="fanuc_green">
       <color rgba="${color_fanuc_green}"/>
     </material>
