Commit message: 20260317

File: support/ros_industrial_support/urdf/assembly_station/assembly_station.urdf.xacro (robot description, xacro)
@@ -2,5 +2,5 @@
 <robot name="assembly_station_urdf" xmlns:xacro="http://www.ros.org/wiki/xacro">
     <xacro:macro name="assembly_station_urdf" params="assembly_station_parent assembly_station_prefix  *origin">
-  <xacro:property name="mesh_path" value="file://$(find ros_industrial_gazebo)"/>
+  <xacro:property name="mesh_path" value="file://$(find ros_industrial_support)"/>
   <joint name="${assembly_station_prefix}joint" type="fixed">
     <xacro:insert_block name="origin" />

File: support/ros_industrial_support/urdf/computer_mobile/computer.urdf.xacro (robot description, xacro)
@@ -2,5 +2,5 @@
 <robot name="computer_urdf" xmlns:xacro="http://www.ros.org/wiki/xacro">
   <xacro:macro name="computer_urdf" params="computer_parent computer_prefix  *origin">
-  <xacro:property name="mesh_path" value="file://$(find ros_industrial_gazebo)"/>
+  <xacro:property name="mesh_path" value="file://$(find ros_industrial_support)"/>
   <joint name="${computer_prefix}joint" type="fixed">
     <xacro:insert_block name="origin" />

File: support/ros_industrial_support/urdf/drop_bin/drop_bin.urdf.xacro (robot description, xacro)
@@ -5,5 +5,5 @@
   <!--<xacro:macro name="bin_urdf" params="prefix mesh_path:='$(find ros_industrial_support)'">-->
   <xacro:macro name="bin_urdf" params="prefix">
-  <xacro:property name="mesh_path" value="file://$(find ros_industrial_gazebo)"/>
+  <xacro:property name="mesh_path" value="file://$(find ros_industrial_support)"/>
     <!-- link list -->
     <link name="${prefix}base_link">

File: support/ros_industrial_support/urdf/part_bin/part_bin.urdf.xacro (robot description, xacro)
@@ -5,5 +5,5 @@
   <!--<xacro:macro name="bin_urdf" params="prefix mesh_path:='$(find ros_industrial_support)'">-->
   <xacro:macro name="bin_urdf" params="prefix">
-  <xacro:property name="mesh_path" value="file://$(find ros_industrial_gazebo)"/>
+  <xacro:property name="mesh_path" value="file://$(find ros_industrial_support)"/>
     <!-- link list -->
     <link name="${prefix}base_link">
