Commit message: 20260317

File: support/ros_industrial_support/urdf/Not Used/shipping_container/shipping_container.urdf.xacro (robot description, xacro)
@@ -14,10 +14,10 @@
       <visual>
         <geometry>
-          <mesh filename="package://ros_industrial_gazebo/models/shipping_container_ariac/meshes/ShippingContainer_Textured.obj" scale="1.3 0.7 1.0"/>
+          <mesh filename="package://ros_industrial_support/models/shipping_container_ariac/meshes/ShippingContainer_Textured.obj" scale="1.3 0.7 1.0"/>
         </geometry>
       </visual>
       <collision>
         <geometry>
-          <mesh filename="package://ros_industrial_gazebo/models/shipping_container_ariac/meshes/ShippingContainer_Textured.obj" scale="1.3 0.7 1.0"/>
+          <mesh filename="package://ros_industrial_support/models/shipping_container_ariac/meshes/ShippingContainer_Textured.obj" scale="1.3 0.7 1.0"/>
         </geometry>
       </collision>

File: support/ros_industrial_support/urdf/Not Used/shipping_container_conveyor/shipping_container_conveyor.urdf.xacro (robot description, xacro)
@@ -14,10 +14,10 @@
       <visual>
         <geometry>
-          <mesh filename="package://ros_industrial_gazebo/models/shipping_container_conveyor_ariac/meshes/ShippingContainer_Textured.obj" scale="1 0.7 1.0"/>
+          <mesh filename="package://ros_industrial_support/models/shipping_container_conveyor_ariac/meshes/ShippingContainer_Textured.obj" scale="1 0.7 1.0"/>
         </geometry>
       </visual>
       <collision>
         <geometry>
-          <mesh filename="package://ros_industrial_gazebo/models/shipping_container_conveyor_ariac/meshes/ShippingContainer_Textured.obj" scale="1 0.7 1.0"/>
+          <mesh filename="package://ros_industrial_support/models/shipping_container_conveyor_ariac/meshes/ShippingContainer_Textured.obj" scale="1 0.7 1.0"/>
         </geometry>
       </collision>

File: support/ros_industrial_support/urdf/Not Used/shipping_container_conveyor_tall/shipping_container_conveyor_tall.urdf.xacro (robot description, xacro)
@@ -14,10 +14,10 @@
       <visual>
         <geometry>
-          <mesh filename="package://ros_industrial_gazebo/models/shipping_container_conveyor_tall_ariac/meshes/ShippingContainer_Textured.obj" scale="0.9 0.7 1.3"/>
+          <mesh filename="package://ros_industrial_support/models/shipping_container_conveyor_tall_ariac/meshes/ShippingContainer_Textured.obj" scale="0.9 0.7 1.3"/>
         </geometry>
       </visual>
       <collision>
         <geometry>
-          <mesh filename="package://ros_industrial_gazebo/models/shipping_container_conveyor_tall_ariac/meshes/ShippingContainer_Textured.obj" scale="0.9 0.7 1.3"/>
+          <mesh filename="package://ros_industrial_support/models/shipping_container_conveyor_tall_ariac/meshes/ShippingContainer_Textured.obj" scale="0.9 0.7 1.3"/>
         </geometry>
       </collision>

File: support/ros_industrial_support/urdf/Not Used/shipping_container_short/shipping_container_short.urdf.xacro (robot description, xacro)
@@ -14,10 +14,10 @@
       <visual>
         <geometry>
-          <mesh filename="package://ros_industrial_gazebo/models/shipping_container_short_ariac/meshes/ShippingContainer_Textured.obj" scale="1.1 0.7 0.8"/>
+          <mesh filename="package://ros_industrial_support/models/shipping_container_short_ariac/meshes/ShippingContainer_Textured.obj" scale="1.1 0.7 0.8"/>
         </geometry>
       </visual>
       <collision>
         <geometry>
-          <mesh filename="package://ros_industrial_gazebo/models/shipping_container_short_ariac/meshes/ShippingContainer_Textured.obj" scale="1.1 0.7 0.8"/>
+          <mesh filename="package://ros_industrial_support/models/shipping_container_short_ariac/meshes/ShippingContainer_Textured.obj" scale="1.1 0.7 0.8"/>
         </geometry>
       </collision>

File: support/ros_industrial_support/urdf/Not Used/yellow_bin/yellow_bin.urdf.xacro (robot description, xacro)
@@ -14,10 +14,10 @@
       <visual>
         <geometry>
-          <mesh filename="package://ros_industrial_gazebo/models/yellow_bin_ariac/meshes/yellow_bin.obj" scale="1 2 1"/>
+          <mesh filename="package://ros_industrial_support/models/yellow_bin_ariac/meshes/yellow_bin.obj" scale="1 2 1"/>
         </geometry>
       </visual>
       <collision>
         <geometry>
-          <mesh filename="package://ros_industrial_gazebo/models/yellow_bin_ariac/meshes/yellow_bin.obj" scale="1 2 1"/>
+          <mesh filename="package://ros_industrial_support/models/yellow_bin_ariac/meshes/yellow_bin.obj" scale="1 2 1"/>
         </geometry>
       </collision>
